File: design_sources/KiCAD/controller_mainboard/emf_arrestor.kicad_sch (KiCad schematic)
At the start: 0 parts

Commit message: Continued development on the schematic. Pins wired. TODO validate.
Other:
- company: Kestech -> Mete Han Keskin
Changed lines of the file:
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@@
 		(date "2025-03-01")
 		(rev "V1.0")
-		(company "Kestech")
-		(comment 1 "MIT License. Copyright (c) 2025 Kestech Fontys")
+		(company "Mete Han Keskin")
+		(comment 1 "MIT License. Copyright (c) 2025 kestech.net")
 	)
 )
