File: design_sources/KiCAD/controller_mainboard/controller_mainboard.kicad_pcb (KiCad board)
At the start: 2 copper layers, 0 parts

Commit message: Adjusted gitignore to ignore backups, removed backup files
Parts:
- added C1: 50V 22pF C0G, Capacitor_SMD:C_0402_1005Metric, F.Cu at (182.8, 76.0)
- added C10: 50V 22pF C0G, Capacitor_SMD:C_0402_1005Metric, F.Cu at (129.2, 182.7)
- added C11: 50V 100nF X7R, Capacitor_SMD:C_0603_1608Metric, F.Cu at (129.7, 163.5)
- added C12: 50V 1uF X5R, Capacitor_SMD:C_0603_1608Metric, F.Cu at (129.7, 166.0)
- added C13: 50V 100nF X7R, Capacitor_SMD:C_0603_1608Metric, F.Cu at (129.7, 168.5)
- added C14: 50V 1uF X5R, Capacitor_SMD:C_0603_1608Metric, F.Cu at (129.7, 171.0)
- added C15: 50V 100nF X7R, Capacitor_SMD:C_0603_1608Metric, F.Cu at (129.7, 173.5)
- added C16: 50V 1uF X5R, Capacitor_SMD:C_0603_1608Metric, F.Cu at (-13.0, 128.0)
- added C17: 50V 100nF X7R, Capacitor_SMD:C_0603_1608Metric, F.Cu at (-13.0, 130.5)
- added C18: 50V 1uF X5R, Capacitor_SMD:C_0603_1608Metric, F.Cu at (-50.7, 139.2)
- added C19: 50V 1uF X5R, Capacitor_SMD:C_0603_1608Metric, F.Cu at (-50.7, 141.7)
- added C2: 50V 22pF C0G, Capacitor_SMD:C_0402_1005Metric, F.Cu at (182.8, 78.0)
- added C20: 50V 1uF X5R, Capacitor_SMD:C_0603_1608Metric, F.Cu at (-50.7, 144.2)
- added C21: 50V 1uF X5R, Capacitor_SMD:C_0603_1608Metric, F.Cu at (-50.7, 146.7)
- added C22: 50V 1uF X5R, Capacitor_SMD:C_0603_1608Metric, F.Cu at (-92.9, 141.0)
- added C23: 50V 100nF X7R, Capacitor_SMD:C_0603_1608Metric, F.Cu at (-48.5, 162.8)
- added C24: 50V 1uF X5R, Capacitor_SMD:C_0603_1608Metric, F.Cu at (-86.3, 157.5)
- added C25: 50V 1uF X5R, Capacitor_SMD:C_0603_1608Metric, F.Cu at (-86.3, 160.0)
- added C26: 50V 100nF X7R, Capacitor_SMD:C_0603_1608Metric, F.Cu at (-46.7, 141.7)
- added C27: 50V 100uF, Capacitor_SMD:CP_Elec_8x10.5, F.Cu at (-84.5, 168.0)
- added C28: 50V 100nF X7R, Capacitor_SMD:C_0603_1608Metric, F.Cu at (-46.7, 144.2)
- added C29: 50V 1uF X5R, Capacitor_SMD:C_0603_1608Metric, F.Cu at (120.7, 182.9)
- added C3: 50V 100nF X7R, Capacitor_SMD:C_0603_1608Metric, F.Cu at (171.3, 66.2)
- added C30: 50V 100uF, Capacitor_SMD:CP_Elec_8x10.5, F.Cu at (109.1, 167.2)
- added C31: 50V 100nF X7R, Capacitor_SMD:C_0603_1608Metric, F.Cu at (120.7, 185.4)
- added C32: 50V 1uF X5R, Capacitor_SMD:C_0603_1608Metric, F.Cu at (120.7, 187.9)
- added C33: 50V 100uF, Capacitor_SMD:CP_Elec_8x10.5, F.Cu at (109.1, 177.3)
- added C34: 50V 100uF, Capacitor_SMD:CP_Elec_8x10.5, F.Cu at (109.1, 187.3)
- added C35: 50V 1uF X5R, Capacitor_SMD:C_0603_1608Metric, F.Cu at (120.6, 81.3)
- added C36: 50V 100nF X7R, Capacitor_SMD:C_0603_1608Metric, F.Cu at (120.6, 83.8)
- added C37: 50V 1uF X5R, Capacitor_SMD:C_0603_1608Metric, F.Cu at (120.6, 86.3)
- added C38: 50V 1uF X5R, Capacitor_SMD:C_0603_1608Metric, F.Cu at (120.6, 88.8)
- added C39: 50V 1uF X5R, Capacitor_SMD:C_0603_1608Metric, F.Cu at (120.6, 91.3)
- added C4: 50V 100uF, Capacitor_SMD:CP_Elec_8x10.5, F.Cu at (180.0, 70.0)
- added C40: 50V 1uF X5R, Capacitor_SMD:C_0603_1608Metric, F.Cu at (120.6, 93.8)
- added C41: 50V 1uF X5R, Capacitor_SMD:C_0603_1608Metric, F.Cu at (120.6, 96.3)
- added C42: 50V 100nF X7R, Capacitor_SMD:C_0603_1608Metric, F.Cu at (124.6, 81.3)
- added C43: 50V 1uF X5R, Capacitor_SMD:C_0603_1608Metric, F.Cu at (124.6, 83.8)
- added C44: 50V 1uF X5R, Capacitor_SMD:C_0603_1608Metric, F.Cu at (124.6, 86.3)
- added C45: 50V 100nF X7R, Capacitor_SMD:C_0603_1608Metric, F.Cu at (124.6, 88.8)
- added C46: 50V 100uF, Capacitor_SMD:CP_Elec_8x10.5, F.Cu at (137.3, 85.0)
- added C47: 50V 100nF X7R, Capacitor_SMD:C_0603_1608Metric, F.Cu at (124.6, 91.3)
- added C48: 50V 1uF X5R, Capacitor_SMD:C_0603_1608Metric, F.Cu at (104.4, 143.9)
- added C49: 50V 100nF X7R, Capacitor_SMD:C_0603_1608Metric, F.Cu at (104.4, 146.4)
- added C5: 50V 100nF X7R, Capacitor_SMD:C_0603_1608Metric, F.Cu at (171.3, 68.7)
- added C50: 50V 1uF X5R, Capacitor_SMD:C_0603_1608Metric, F.Cu at (104.4, 148.9)
- added C51: 50V 1uF X5R, Capacitor_SMD:C_0603_1608Metric, F.Cu at (104.4, 151.4)
- added C52: 50V 1uF X5R, Capacitor_SMD:C_0603_1608Metric, F.Cu at (104.4, 153.9)
- added C53: 50V 1uF X5R, Capacitor_SMD:C_0603_1608Metric, F.Cu at (104.4, 156.4)
- added C54: 50V 1uF X5R, Capacitor_SMD:C_0603_1608Metric, F.Cu at (104.4, 159.0)
- added C55: 50V 100nF X7R, Capacitor_SMD:C_0603_1608Metric, F.Cu at (108.4, 143.9)
- added C56: 50V 1uF X5R, Capacitor_SMD:C_0603_1608Metric, F.Cu at (108.4, 146.4)
- added C57: 50V 1uF X5R, Capacitor_SMD:C_0603_1608Metric, F.Cu at (108.4, 148.9)
- added C58: 50V 100nF X7R, Capacitor_SMD:C_0603_1608Metric, F.Cu at (108.4, 151.4)
- added C59: 50V 100uF, Capacitor_SMD:CP_Elec_8x10.5, F.Cu at (121.1, 147.7)
- added C6: 50V 100nF X7R, Capacitor_SMD:C_0603_1608Metric, F.Cu at (171.3, 71.2)
- added C60: 50V 100nF X7R, Capacitor_SMD:C_0603_1608Metric, F.Cu at (108.4, 153.9)
- added C61: 50V 1uF X5R, Capacitor_SMD:C_0603_1608Metric, F.Cu at (155.1, 143.9)
- added C62: 50V 100nF X7R, Capacitor_SMD:C_0603_1608Metric, F.Cu at (155.1, 146.4)
- added C63: 50V 1uF X5R, Capacitor_SMD:C_0603_1608Metric, F.Cu at (155.1, 148.9)
- added C64: 50V 1uF X5R, Capacitor_SMD:C_0603_1608Metric, F.Cu at (155.1, 151.4)
- added C65: 50V 1uF X5R, Capacitor_SMD:C_0603_1608Metric, F.Cu at (155.1, 153.9)
- added C66: 50V 1uF X5R, Capacitor_SMD:C_0603_1608Metric, F.Cu at (155.1, 156.4)
- added C67: 50V 1uF X5R, Capacitor_SMD:C_0603_1608Metric, F.Cu at (155.1, 159.0)
- added C68: 50V 100nF X7R, Capacitor_SMD:C_0603_1608Metric, F.Cu at (159.1, 143.9)
- added C69: 50V 1uF X5R, Capacitor_SMD:C_0603_1608Metric, F.Cu at (159.1, 146.4)
- added C7: 50V 1uF X5R, Capacitor_SMD:C_0603_1608Metric, F.Cu at (171.3, 73.7)
- added C70: 50V 1uF X5R, Capacitor_SMD:C_0603_1608Metric, F.Cu at (159.1, 148.9)
- added C71: 50V 100nF X7R, Capacitor_SMD:C_0603_1608Metric, F.Cu at (159.1, 151.4)
- added C72: 50V 100uF, Capacitor_SMD:CP_Elec_8x10.5, F.Cu at (171.8, 147.7)
- added C73: 50V 100nF X7R, Capacitor_SMD:C_0603_1608Metric, F.Cu at (159.1, 153.9)
- added C74: N.C., Capacitor_SMD:C_0603_1608Metric, F.Cu at (53.8, 163.5)
- added C75: N.C., Capacitor_SMD:C_0603_1608Metric, F.Cu at (53.8, 166.0)
- added C76: N.C., Capacitor_SMD:C_0603_1608Metric, F.Cu at (53.8, 175.5)
- added C77: N.C., Capacitor_SMD:C_0603_1608Metric, F.Cu at (53.8, 178.0)
- added C78: N.C., Capacitor_SMD:C_0603_1608Metric, F.Cu at (171.3, 83.3)
- added C79: N.C., Capacitor_SMD:C_0603_1608Metric, F.Cu at (171.3, 85.8)
- added C8: 50V 100nF X7R, Capacitor_SMD:C_0603_1608Metric, F.Cu at (171.3, 76.2)
- added C80: N.C., Capacitor_SMD:C_0603_1608Metric, F.Cu at (171.3, 95.3)
- added C81: N.C., Capacitor_SMD:C_0603_1608Metric, F.Cu at (171.3, 97.8)
- added C82: N.C., Capacitor_SMD:C_0603_1608Metric, F.Cu at (129.7, 176.0)
- added C83: N.C., Capacitor_SMD:C_0603_1608Metric, F.Cu at (-97.0, 170.0)
- added C84: N.C., Capacitor_SMD:C_0603_1608Metric, F.Cu at (124.6, 93.8)
- added C85: N.C., Capacitor_SMD:C_0603_1608Metric, F.Cu at (108.4, 156.4)
- added C86: N.C., Capacitor_SMD:C_0603_1608Metric, F.Cu at (159.1, 156.4)
- added C87: N.C., Capacitor_SMD:C_0603_1608Metric, F.Cu at (-107.5, 170.0)
- added C88: N.C., Capacitor_SMD:C_0603_1608Metric, F.Cu at (124.6, 96.3)
- added C89: N.C., Capacitor_SMD:C_0603_1608Metric, F.Cu at (108.4, 159.0)
- added C9: 50V 22pF C0G, Capacitor_SMD:C_0402_1005Metric, F.Cu at (129.2, 180.8)
- added C90: N.C., Capacitor_SMD:C_0603_1608Metric, F.Cu at (159.1, 159.0)
- added C91: 50V 100nF X7R, Capacitor_SMD:C_0603_1608Metric, F.Cu at (73.5, 78.6)
- added D1: LED RED, LED_SMD:LED_0603_1608Metric, F.Cu at (114.5, 91.7)
- added D10: 40V 5A, Diode_SMD:D_SMA, F.Cu at (-96.1, 184.6)
- added D11: 40V 5A, Diode_SMD:D_SMA, F.Cu at (-107.6, 185.6)
- added D12: 40V 5A, Diode_SMD:D_SMA, F.Cu at (-97.0, 163.0)
- added D13: 40V 5A, Diode_SMD:D_SMA, F.Cu at (-106.5, 162.5)
- added D14: 40V 5A, Diode_SMD:D_SMA, F.Cu at (119.8, 179.4)
- added D15: 40V 5A, Diode_SMD:D_SMA, F.Cu at (154.8, 70.5)
- added D16: 40V 5A, Diode_SMD:D_SMA, F.Cu at (154.8, 75.1)
- added D17: LED GREEN, LED_SMD:LED_0805_2012Metric, F.Cu at (146.2, 86.2)
- added D18: 40V 5A, Diode_SMD:D_SMA, F.Cu at (154.8, 79.6)
- added D19: 40V 5A, Diode_SMD:D_SMA, F.Cu at (154.8, 84.2)
- added D2: 40V 5A, Diode_SMD:D_SMA, F.Cu at (111.7, 101.9)
- added D20: 40V 5A, Diode_SMD:D_SMA, F.Cu at (154.8, 88.7)
- added D21: 40V 5A, Diode_SMD:D_SMA, F.Cu at (154.8, 93.3)
- added D22: 40V 5A, Diode_SMD:D_SMA, F.Cu at (138.6, 133.2)
- added D23: 40V 5A, Diode_SMD:D_SMA, F.Cu at (138.6, 137.7)
- added D24: LED GREEN, LED_SMD:LED_0805_2012Metric, F.Cu at (130.1, 148.8)
- added D25: 40V 5A, Diode_SMD:D_SMA, F.Cu at (138.6, 142.3)
- added D26: 40V 5A, Diode_SMD:D_SMA, F.Cu at (138.6, 146.8)
- added D27: 40V 5A, Diode_SMD:D_SMA, F.Cu at (138.6, 151.4)
- added D28: 40V 5A, Diode_SMD:D_SMA, F.Cu at (138.6, 155.9)
- added D29: 40V 5A, Diode_SMD:D_SMA, F.Cu at (189.3, 133.2)
- added D3: 40V 5A, Diode_SMD:D_SMA, F.Cu at (177.3, 77.3)
- added D30: 40V 5A, Diode_SMD:D_SMA, F.Cu at (189.3, 137.7)
- added D31: LED GREEN, LED_SMD:LED_0805_2012Metric, F.Cu at (180.7, 148.8)
- added D32: 40V 5A, Diode_SMD:D_SMA, F.Cu at (189.3, 142.3)
- added D33: 40V 5A, Diode_SMD:D_SMA, F.Cu at (189.3, 146.8)
- added D34: 40V 5A, Diode_SMD:D_SMA, F.Cu at (189.3, 151.4)
- added D35: 40V 5A, Diode_SMD:D_SMA, F.Cu at (189.3, 155.9)
- added D36: LED GREEN, LED_SMD:LED_0805_2012Metric, F.Cu at (109.8, 105.7)
- added D4: LED YELLOW, LED_SMD:LED_0603_1608Metric, F.Cu at (145.6, 163.5)
- added D5: LED YELLOW, LED_SMD:LED_0603_1608Metric, F.Cu at (145.6, 166.1)
- added D6: 40V 5A, Diode_SMD:D_SMA, F.Cu at (143.3, 181.5)
- added D7: 40V 5A, Diode_SMD:D_SMA, F.Cu at (-20.0, 133.0)
- added D8: 40V 5A, Diode_SMD:D_SMA, F.Cu at (-0.50, 144.5)
- added D9: LED GREEN, LED_SMD:LED_0805_2012Metric, F.Cu at (-99.6, 136.0)
- added F1: Fuse 20A, Custom_feetprint:BLX-A fuse holder, F.Cu at (91.4, 96.3)
- added F2: 5A, Custom_feetprint:BLX-A fuse holder, F.Cu at (-82.5, 135.8)
- added F3: 5A, Custom_feetprint:BLX-A fuse holder, F.Cu at (134.6, 74.2)
- added F4: 5A, Custom_feetprint:BLX-A fuse holder, F.Cu at (118.4, 136.8)
- added F5: 5A, Custom_feetprint:BLX-A fuse holder, F.Cu at (169.1, 136.8)
- added FB1: GZ2012D101TF, Inductor_SMD:L_0805_2012Metric, F.Cu at (114.3, 105.6)
- added J1: XT-90, Custom_feetprint:XT-90_Connector, F.Cu at (87.5, 83.9)
- added J10: 01x08_2.54mm _socket, Connector_PinSocket_2.54mm:PinSocket_1x08_P2.54mm_Vertical, F.Cu at (114.3, 48.9)
- added J11: 2P_screw_term, Connector_JST:JST_NV_B02P-NV_1x02_P5.00mm_Vertical, F.Cu at (-116.5, 172.5)
- added J12: 2P_screw_term, Connector_JST:JST_NV_B02P-NV_1x02_P5.00mm_Vertical, F.Cu at (62.9, 61.9)
- added J13: 2P_screw_term, Connector_JST:JST_NV_B02P-NV_1x02_P5.00mm_Vertical, F.Cu at (62.9, 72.4)
- added J14: 2P_screw_term, Connector_JST:JST_NV_B02P-NV_1x02_P5.00mm_Vertical, F.Cu at (62.9, 83.0)
- added J16: 02x03_pinheader, Connector_PinHeader_2.54mm:PinHeader_2x03_P2.54mm_Vertical, F.Cu at (189.0, 67.3)
- added J17: 01x05_Socket, Connector_PinSocket_2.54mm:PinSocket_1x05_P2.54mm_Vertical, F.Cu at (134.1, 164.5)
- added J19: 02x03_pinheader, Connector_PinHeader_2.54mm:PinHeader_2x03_P2.54mm_Vertical, F.Cu at (138.7, 164.5)
- added J2: XT-60, Connector_AMASS:AMASS_XT60-M_1x02_P7.20mm_Vertical, F.Cu at (76.6, 51.7)
- added J20: 01x04_JST_PH, Connector_JST:JST_PH_B4B-PH-K_1x04_P2.00mm_Vertical, F.Cu at (58.8, 164.9)
- added J21: 01x04_JST_PH, Connector_JST:JST_PH_B4B-PH-K_1x04_P2.00mm_Vertical, F.Cu at (58.8, 177.0)
- added J22: 01x04_JST_PH, Connector_JST:JST_PH_B4B-PH-K_1x04_P2.00mm_Vertical, F.Cu at (176.3, 84.7)
- added J23: 01x04_JST_PH, Connector_JST:JST_PH_B4B-PH-K_1x04_P2.00mm_Vertical, F.Cu at (176.3, 96.8)
- added J24: XT-60, Connector_AMASS:AMASS_XT60-M_1x02_P7.20mm_Vertical, F.Cu at (76.6, 62.0)
- added J25: XT-60, Connector_AMASS:AMASS_XT60-M_1x02_P7.20mm_Vertical, F.Cu at (76.6, 72.2)
- added J3: USB_C_Receptacle_USB2.0_16P, Connector_USB:USB_C_Receptacle_GCT_USB4105-xx-A_16P_TopMnt_Horizontal, F.Cu at (105.4, 82.6)
- added J4: 01x08_2.54mm _socket, Connector_PinSocket_2.54mm:PinSocket_1x08_P2.54mm_Vertical, F.Cu at (95.9, 48.9)
- added J5: 01x08_2.54mm _socket, Connector_PinSocket_2.54mm:PinSocket_1x08_P2.54mm_Vertical, F.Cu at (100.5, 48.9)
- added J6: 01x08_2.54mm _socket, Connector_PinSocket_2.54mm:PinSocket_1x08_P2.54mm_Vertical, F.Cu at (105.1, 48.9)
- added J7: 02x18_2.54mm_socket, Connector_PinHeader_2.54mm:PinHeader_2x18_P2.54mm_Vertical, F.Cu at (54.1, 48.9)
- added J8: Conn_01x10_2.54mm_socket, Connector_PinSocket_2.54mm:PinSocket_1x10_P2.54mm_Vertical, F.Cu at (91.3, 48.9)
- added J9: 01x08_2.54mm _socket, Connector_PinSocket_2.54mm:PinSocket_1x08_P2.54mm_Vertical, F.Cu at (109.7, 48.9)
- added JP1: SolderJumper_2_Open, Jumper:SolderJumper-2_P1.3mm_Open_RoundedPad1.0x1.5mm, F.Cu at (133.9, 178.7)
- added L1: 15mA 10uH 1.15Ohm, Inductor_SMD:L_0805_2012Metric, F.Cu at (196.1, 76.2)
- added L10: 5A 1uH, Inductor_SMD:L_APV_ANR5040, F.Cu at (196.6, 140.8)
- added L2: 5A 1uH, Inductor_SMD:L_APV_ANR5040, F.Cu at (-93.0, 158.0)
- added L3: 5A 1uH, Inductor_SMD:L_APV_ANR5040, F.Cu at (-99.0, 158.0)
- added L4: 3A 15uH, Inductor_SMD:L_APV_APH0630, F.Cu at (120.8, 166.3)
- added L5: 5A 1uH, Inductor_SMD:L_APV_ANR5040, F.Cu at (162.1, 71.6)
- added L6: 5A 1uH, Inductor_SMD:L_APV_ANR5040, F.Cu at (162.1, 78.2)
- added L7: 5A 1uH, Inductor_SMD:L_APV_ANR5040, F.Cu at (146.0, 134.2)
- added L8: 5A 1uH, Inductor_SMD:L_APV_ANR5040, F.Cu at (146.0, 140.8)
- added L9: 5A 1uH, Inductor_SMD:L_APV_ANR5040, F.Cu at (196.6, 134.2)
- added Q1: 2N7002, Package_TO_SOT_SMD:SOT-23, F.Cu at (110.0, 92.8)
- added Q10: IRF3205, Package_TO_SOT_THT:TO-220F-3_Horizontal_TabDown, F.Cu at (157.4, 66.5)
- added Q11: IRF3205, Package_TO_SOT_THT:TO-220F-3_Horizontal_TabDown, F.Cu at (105.8, 129.1)
- added Q12: IRF3205, Package_TO_SOT_THT:TO-220F-3_Horizontal_TabDown, F.Cu at (117.6, 129.1)
- added Q13: IRF3205, Package_TO_SOT_THT:TO-220F-3_Horizontal_TabDown, F.Cu at (129.4, 129.1)
- added Q14: IRF3205, Package_TO_SOT_THT:TO-220F-3_Horizontal_TabDown, F.Cu at (141.2, 129.1)
- added Q15: IRF3205, Package_TO_SOT_THT:TO-220F-3_Horizontal_TabDown, F.Cu at (156.5, 129.1)
- added Q16: IRF3205, Package_TO_SOT_THT:TO-220F-3_Horizontal_TabDown, F.Cu at (168.3, 129.1)
- added Q17: IRF3205, Package_TO_SOT_THT:TO-220F-3_Horizontal_TabDown, F.Cu at (180.1, 129.1)
- added Q18: IRF3205, Package_TO_SOT_THT:TO-220F-3_Horizontal_TabDown, F.Cu at (191.9, 129.1)
- added Q3: IRF3205, Package_TO_SOT_THT:TO-220F-3_Horizontal_TabDown, B.Cu at (-92.5, 190.6)
- added Q4: IRF3205, Package_TO_SOT_THT:TO-220F-3_Horizontal_TabDown, B.Cu at (-103.5, 190.6)
- added Q5: IRF3205, Package_TO_SOT_THT:TO-220F-3_Horizontal_TabDown, B.Cu at (-92.5, 167.0)
- added Q6: IRF3205, Package_TO_SOT_THT:TO-220F-3_Horizontal_TabDown, B.Cu at (-103.5, 167.1)
- added Q7: IRF3205, Package_TO_SOT_THT:TO-220F-3_Horizontal_TabDown, F.Cu at (122.0, 66.5)
- added Q8: IRF3205, Package_TO_SOT_THT:TO-220F-3_Horizontal_TabDown, F.Cu at (133.8, 66.5)
- added Q9: IRF3205, Package_TO_SOT_THT:TO-220F-3_Horizontal_TabDown, F.Cu at (145.6, 66.5)
- added R1: 10k 63mW, Resistor_SMD:R_0402_1005Metric, F.Cu at (112.7, 78.3)
- added R10: 10k 63mW, Resistor_SMD:R_0402_1005Metric, F.Cu at (195.3, 65.9)
- added R11: 1M 63mW, Resistor_SMD:R_0603_1608Metric, F.Cu at (129.7, 178.5)
- added R12: 1k 63mW, Resistor_SMD:R_0402_1005Metric, F.Cu at (137.8, 172.9)
- added R13: 1k 63mW, Resistor_SMD:R_0402_1005Metric, F.Cu at (137.8, 174.9)
- added R14: 1k 63mW, Resistor_SMD:R_0402_1005Metric, F.Cu at (137.8, 176.9)
- added R15: 1k 63mW, Resistor_SMD:R_0402_1005Metric, F.Cu at (137.8, 178.9)
- added R16: 1k 63mW, Resistor_SMD:R_0402_1005Metric, F.Cu at (137.8, 180.9)
- added R17: 10k 63mW, Resistor_SMD:R_0402_1005Metric, F.Cu at (137.8, 182.9)
- added R18: 10k 63mW, Resistor_SMD:R_0402_1005Metric, F.Cu at (-39.2, 144.0)
- added R19: 10k 63mW, Resistor_SMD:R_0402_1005Metric, F.Cu at (-39.2, 146.0)
- added R20: 10k 63mW, Resistor_SMD:R_0402_1005Metric, F.Cu at (-39.2, 148.0)
- added R21: N.C., Resistor_SMD:R_0402_1005Metric, F.Cu at (-36.3, 144.0)
- added R22: 1k 63mW, Resistor_SMD:R_0402_1005Metric, F.Cu at (-97.0, 141.5)
- added R23: 1k 63mW, Resistor_SMD:R_0402_1005Metric, F.Cu at (-40.5, 165.0)
- added R24: 1k 63mW, Resistor_SMD:R_0402_1005Metric, F.Cu at (-40.5, 162.0)
- added R25: 50m 750mW 1%, Resistor_SMD:R_2512_6332Metric, F.Cu at (-35.5, 163.5)
- added R26: 10k 63mW, Resistor_SMD:R_0402_1005Metric, F.Cu at (117.2, 182.7)
- added R27: 10k 63mW, Resistor_SMD:R_0402_1005Metric, F.Cu at (117.2, 184.6)
- added R28: 10k 63mW, Resistor_SMD:R_0402_1005Metric, F.Cu at (117.2, 186.6)
- added R29: 10k 63mW, Resistor_SMD:R_0402_1005Metric, F.Cu at (117.2, 188.6)
- added R30: 10k 63mW, Resistor_SMD:R_0402_1005Metric, F.Cu at (132.1, 91.1)
- added R31: 10k 63mW, Resistor_SMD:R_0402_1005Metric, F.Cu at (132.1, 93.0)
- added R32: 10k 63mW, Resistor_SMD:R_0402_1005Metric, F.Cu at (132.1, 95.0)
- added R33: N.C., Resistor_SMD:R_0402_1005Metric, F.Cu at (135.0, 91.1)
- added R34: 1k 63mW, Resistor_SMD:R_0402_1005Metric, F.Cu at (135.0, 93.0)
- added R35: 1k 63mW, Resistor_SMD:R_0402_1005Metric, F.Cu at (135.0, 95.0)
- added R36: 1k 63mW, Resistor_SMD:R_0402_1005Metric, F.Cu at (137.9, 91.1)
- added R37: 50m 750mW 1%, Resistor_SMD:R_2512_6332Metric, F.Cu at (143.7, 92.5)
- added R38: 10k 63mW, Resistor_SMD:R_0402_1005Metric, F.Cu at (115.9, 153.7)
- added R39: 10k 63mW, Resistor_SMD:R_0402_1005Metric, F.Cu at (115.9, 155.7)
- added R4: 1k 63mW, Resistor_SMD:R_0402_1005Metric, F.Cu at (112.7, 80.3)
- added R40: 10k 63mW, Resistor_SMD:R_0402_1005Metric, F.Cu at (115.9, 157.7)
- added R41: N.C., Resistor_SMD:R_0402_1005Metric, F.Cu at (118.8, 153.7)
- added R42: 1k 63mW, Resistor_SMD:R_0402_1005Metric, F.Cu at (118.8, 155.7)
- added R43: 1k 63mW, Resistor_SMD:R_0402_1005Metric, F.Cu at (118.8, 157.7)
- added R44: 1k 63mW, Resistor_SMD:R_0402_1005Metric, F.Cu at (121.7, 153.7)
- added R45: 50m 750mW 1%, Resistor_SMD:R_2512_6332Metric, F.Cu at (127.5, 155.1)
- added R46: 10k 63mW, Resistor_SMD:R_0402_1005Metric, F.Cu at (166.6, 153.7)
- added R47: 10k 63mW, Resistor_SMD:R_0402_1005Metric, F.Cu at (166.6, 155.7)
- added R48: 10k 63mW, Resistor_SMD:R_0402_1005Metric, F.Cu at (166.6, 157.7)
- added R49: N.C., Resistor_SMD:R_0402_1005Metric, F.Cu at (169.5, 153.7)
- added R5: 5.1K 100mW, Capacitor_SMD:C_0603_1608Metric, F.Cu at (73.5, 81.1)
- added R50: 1k 63mW, Resistor_SMD:R_0402_1005Metric, F.Cu at (169.5, 155.7)
- added R51: 1k 63mW, Resistor_SMD:R_0402_1005Metric, F.Cu at (169.5, 157.7)
- added R52: 1k 63mW, Resistor_SMD:R_0402_1005Metric, F.Cu at (172.4, 153.7)
- added R53: 50m 750mW 1%, Resistor_SMD:R_2512_6332Metric, F.Cu at (178.2, 155.1)
- added R54: 5.1K 100mW, Capacitor_SMD:C_0603_1608Metric, F.Cu at (53.8, 168.5)
- added R55: 5.1K 100mW, Capacitor_SMD:C_0603_1608Metric, F.Cu at (53.8, 171.0)
- added R56: 5.1K 100mW, Capacitor_SMD:C_0603_1608Metric, F.Cu at (53.8, 180.5)
- added R57: 5.1K 100mW, Capacitor_SMD:C_0603_1608Metric, F.Cu at (53.8, 183.0)
- added R58: 5.1K 100mW, Capacitor_SMD:C_0603_1608Metric, F.Cu at (171.3, 88.3)
- added R59: 5.1K 100mW, Capacitor_SMD:C_0603_1608Metric, F.Cu at (171.3, 90.8)
- added R6: 5.1K 100mW, Capacitor_SMD:C_0603_1608Metric, F.Cu at (73.5, 83.6)
- added R60: 5.1K 100mW, Capacitor_SMD:C_0603_1608Metric, F.Cu at (171.3, 100.3)
- added R61: 5.1K 100mW, Capacitor_SMD:C_0603_1608Metric, F.Cu at (171.3, 102.8)
- added R62: 1k 63mW, Resistor_SMD:R_0402_1005Metric, F.Cu at (112.7, 82.3)
- added R63: 1k 63mW, Resistor_SMD:R_0402_1005Metric, F.Cu at (112.7, 84.3)
- added R64: 0R 100mW, Resistor_SMD:R_0603_1608Metric, F.Cu at (-69.7, 173.5)
- added R65: 0R 100mW, Resistor_SMD:R_0603_1608Metric, F.Cu at (128.6, 81.3)
- added R66: 0R 100mW, Resistor_SMD:R_0603_1608Metric, F.Cu at (112.5, 143.9)
- added R67: 0R 100mW, Resistor_SMD:R_0603_1608Metric, F.Cu at (163.1, 143.9)
- added R68: 0R 100mW, Resistor_SMD:R_0603_1608Metric, F.Cu at (-71.2, 170.5)
- added R69: 0R 100mW, Resistor_SMD:R_0603_1608Metric, F.Cu at (128.6, 83.8)
- added R7: 22R 100mW, Resistor_SMD:R_0603_1608Metric, F.Cu at (73.5, 86.1)
- added R70: 0R 100mW, Resistor_SMD:R_0603_1608Metric, F.Cu at (112.5, 146.4)
- added R71: 0R 100mW, Resistor_SMD:R_0603_1608Metric, F.Cu at (163.1, 146.4)
- added R72: 0R 100mW, Resistor_SMD:R_0603_1608Metric, F.Cu at (-71.5, 164.0)
- added R73: 0R 100mW, Resistor_SMD:R_0603_1608Metric, F.Cu at (128.6, 86.3)
- added R74: 0R 100mW, Resistor_SMD:R_0603_1608Metric, F.Cu at (112.5, 148.9)
- added R75: 0R 100mW, Resistor_SMD:R_0603_1608Metric, F.Cu at (163.1, 148.9)
- added R76: 0R 100mW, Resistor_SMD:R_0603_1608Metric, F.Cu at (-71.3, 167.5)
- added R77: 0R 100mW, Resistor_SMD:R_0603_1608Metric, F.Cu at (128.6, 88.8)
- added R78: 0R 100mW, Resistor_SMD:R_0603_1608Metric, F.Cu at (112.5, 151.4)
- added R79: 0R 100mW, Resistor_SMD:R_0603_1608Metric, F.Cu at (163.1, 151.4)
- added R8: 22R 100mW, Resistor_SMD:R_0603_1608Metric, F.Cu at (73.5, 88.6)
- added R80: 5.1K 100mW, Capacitor_SMD:C_0603_1608Metric, F.Cu at (73.5, 91.2)
- added R81: 10k 63mW, Resistor_SMD:R_0402_1005Metric, F.Cu at (112.7, 86.3)
- added R82: 10k 63mW, Resistor_SMD:R_0402_1005Metric, F.Cu at (-18.0, 145.5)
- added R83: 10k 63mW, Resistor_SMD:R_0402_1005Metric, F.Cu at (137.9, 93.0)
- added R84: 10k 63mW, Resistor_SMD:R_0402_1005Metric, F.Cu at (121.7, 155.7)
- added R85: 10k 63mW, Resistor_SMD:R_0402_1005Metric, F.Cu at (172.4, 155.7)
- added R86: 10k 63mW, Resistor_SMD:R_0402_1005Metric, F.Cu at (-18.5, 140.5)
- added R87: 10k 63mW, Resistor_SMD:R_0402_1005Metric, F.Cu at (137.9, 95.0)
- added R88: 10k 63mW, Resistor_SMD:R_0402_1005Metric, F.Cu at (121.7, 157.7)
- added R89: 10k 63mW, Resistor_SMD:R_0402_1005Metric, F.Cu at (172.4, 157.7)
- added R9: 1M 63mW, Resistor_SMD:R_0603_1608Metric, F.Cu at (171.3, 78.8)
- added R90: 10k 63mW, Resistor_SMD:R_0402_1005Metric, F.Cu at (195.3, 67.9)
- added R91: 10k 63mW, Resistor_SMD:R_0402_1005Metric, F.Cu at (195.3, 69.9)
- added SW1: SW_Push, Button_Switch_SMD:SW_SPST_PTS645, F.Cu at (208.0, 53.8)
- added U1: ATmega2560-16A, Package_QFP:TQFP-100_14x14mm_P0.5mm, F.Cu at (178.4, 55.8)
- added U10: HIP4082IBZT, Package_SO:SOIC-16_3.9x9.9mm_P1.27mm, F.Cu at (197.5, 150.1)
- added U11: INA180A1IDBVR, Package_TO_SOT_SMD:SOT-23-5, F.Cu at (181.0, 145.0)
- added U12: USBLC6-4SC6, Package_TO_SOT_SMD:SOT-23-6, F.Cu at (110.2, 97.4)
- added U2: ATmega16U2-M, Package_DFN_QFN:QFN-32-1EP_5x5mm_P0.5mm_EP3.1x3.1mm, F.Cu at (142.9, 175.6)
- added U3: HIP4082IBZT, Package_SO:SOIC-16_3.9x9.9mm_P1.27mm, F.Cu at (-8.26, 140.3)
- added U4: INA180A1IDBVR, Package_TO_SOT_SMD:SOT-23-5, F.Cu at (-44.5, 163.0)
- added U5: TPS5430DDA, Package_SO:TI_SO-PowerPAD-8_ThermalVias, F.Cu at (120.1, 173.8)
- added U6: HIP4082IBZT, Package_SO:SOIC-16_3.9x9.9mm_P1.27mm, F.Cu at (163.0, 87.4)
- added U7: INA180A1IDBVR, Package_TO_SOT_SMD:SOT-23-5, F.Cu at (146.6, 82.4)
- added U8: HIP4082IBZT, Package_SO:SOIC-16_3.9x9.9mm_P1.27mm, F.Cu at (146.9, 150.1)
- added U9: INA180A1IDBVR, Package_TO_SOT_SMD:SOT-23-5, F.Cu at (130.4, 145.0)
- added Y1: 16MHz, Crystal:Resonator_SMD_Murata_CSTxExxV-3Pin_3.0x1.1mm, F.Cu at (196.4, 72.7)
- added Y2: 16MHz, Crystal:Resonator_SMD_Murata_CSTxExxV-3Pin_3.0x1.1mm, F.Cu at (146.1, 169.2)
