File: design_sources/KiCAD/controller_mainboard/controller_mainboard.kicad_pcb (KiCad board)
At the start: 2 copper layers, 288 parts, among them J1 XT-90, J10 01x08_2.54mm _socket, J11 2P_screw_term, J12 2P_screw_term, J13 2P_screw_term, J14 2P_screw_term, J16 02x03_pinheader, J17 01x05_Socket, J19 02x03_pinheader, J2 XT-60, J20 01x04_JST_PH, J21 01x04_JST_PH, J22 01x04_JST_PH, J23 01x04_JST_PH, J24 XT-60, J25 XT-60, J3 USB_C_Receptacle_USB2.0_16P, J4 01x08_2.54mm _socket, J5 01x08_2.54mm _socket, J6 01x08_2.54mm _socket, J7 02x18_2.54mm_socket, J8 Conn_01x10_2.54mm_socket, J9 01x08_2.54mm _socket, Q1 2N7002, Q10 IRF3205, Q11 IRF3205, Q12 IRF3205, Q13 IRF3205, Q14 IRF3205, Q15 IRF3205, Q16 IRF3205, Q17 IRF3205, Q18 IRF3205, Q3 IRF3205, Q4 IRF3205, Q5 IRF3205, Q6 IRF3205, Q7 IRF3205, Q8 IRF3205, Q9 IRF3205, SW1 SW_Push, U1 ATmega2560-16A, U10 HIP4082IBZT, U11 INA180A1IDBVR, U12 USBLC6-4SC6, U2 ATmega16U2-M, U3 HIP4082IBZT, U4 INA180A1IDBVR, U5 TPS5430DDA, U6 HIP4082IBZT, U7 INA180A1IDBVR, U8 HIP4082IBZT, U9 INA180A1IDBVR, Y1 16MHz, Y2 16MHz

Commit message: started initial pcb layout
Parts:
- added J18: 02x02_pinheader, Connector_PinHeader_2.54mm:PinHeader_2x02_P2.54mm_Vertical, F.Cu at (217.0, 111.0)
- Q10, Q7, Q8, Q9: footprint Package_TO_SOT_THT:TO-220F-3_Horizontal_TabDown -> Package_TO_SOT_THT:TO-220-3_Horizontal_TabDown; moved to B.Cu
- Q11, Q12, Q13, Q14, Q15, Q16, Q17, Q18, Q3, Q4, Q5, Q6: footprint Package_TO_SOT_THT:TO-220F-3_Horizontal_TabDown -> Package_TO_SOT_THT:TO-220-3_Horizontal_TabDown
- moved U6 262.1 mm to (-71.0, 205.4)
- moved R83 243.6 mm to (-79.0, 204.0), turned to 180 degrees
- moved R87 241.9 mm to (-79.0, 202.0), turned to 180 degrees
- moved D16 241.6 mm to (-66.5, 172.0), turned to 90 degrees
- moved D15 240.4 mm to (-66.5, 164.5), turned to -90 degrees
- moved D19 236.0 mm to (-59.5, 183.0), turned to 180 degrees
- moved Q10 234.6 mm to (-55.0, 166.2), turned to 180 degrees
- moved L5 227.2 mm to (-54.0, 141.5), turned to 90 degrees
- moved D21 224.6 mm to (-59.0, 162.0), turned to 180 degrees
- moved Q8 224.4 mm to (-55.0, 187.9), turned to 180 degrees
- moved C35 219.9 mm to (-46.7, 224.0)
- moved C36 219.9 mm to (-46.7, 226.5)
- moved C37 219.9 mm to (-46.7, 229.0)
- moved C38 219.9 mm to (-46.7, 231.5)
- moved C39 219.9 mm to (-46.7, 234.0)
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Connections:
- C16 pad 1: +BATT -> Net-(D7-A)
- C17 pad 2: +BATT -> Net-(D7-A)
- C22 pad 1: Net-(C22-Pad1) -> Net-(D7-A)
- C35 pad 1: +BATT -> Net-(D15-A)
- C36 pad 2: +BATT -> Net-(D15-A)
- C41 pad 1: Net-(C41-Pad1) -> Net-(D15-A)
- C48 pad 1: +BATT -> Net-(D22-A)
- C49 pad 2: +BATT -> Net-(D22-A)
- C54 pad 1: Net-(C54-Pad1) -> Net-(D22-A)
- C61 pad 1: +BATT -> Net-(D29-A)
- C62 pad 2: +BATT -> Net-(D29-A)
- C67 pad 1: Net-(C67-Pad1) -> Net-(D29-A)
- D15 pad 2: +BATT -> Net-(D15-A)
- D16 pad 2: +BATT -> Net-(D15-A)
- D22 pad 2: +BATT -> Net-(D22-A)
- D23 pad 2: +BATT -> Net-(D22-A)
- D29 pad 2: +BATT -> Net-(D29-A)
- D30 pad 2: +BATT -> Net-(D29-A)
- D7 pad 2: +BATT -> Net-(D7-A)
- D8 pad 2: +BATT -> Net-(D7-A)
- F2 pad 2: Net-(C22-Pad1) -> Net-(D7-A)
- F3 pad 2: Net-(C41-Pad1) -> Net-(D15-A)
- F4 pad 2: Net-(C54-Pad1) -> Net-(D22-A)
- F5 pad 2: Net-(C67-Pad1) -> Net-(D29-A)
- L10 pad 2: Net-(C67-Pad1) -> Net-(D29-A)
- L2 pad 1: Net-(C22-Pad1) -> Net-(D7-A)
- L3 pad 2: Net-(C22-Pad1) -> Net-(D7-A)
- L5 pad 1: Net-(C41-Pad1) -> Net-(D15-A)
- L6 pad 2: Net-(C41-Pad1) -> Net-(D15-A)
- L7 pad 1: Net-(C54-Pad1) -> Net-(D22-A)
- L8 pad 2: Net-(C54-Pad1) -> Net-(D22-A)
- L9 pad 1: Net-(C67-Pad1) -> Net-(D29-A)
- R22 pad 1: Net-(C22-Pad1) -> Net-(D7-A)
- R34 pad 1: Net-(C41-Pad1) -> Net-(D15-A)
- R42 pad 1: Net-(C54-Pad1) -> Net-(D22-A)
- R50 pad 1: Net-(C67-Pad1) -> Net-(D29-A)
- U10 pad 12: +BATT -> Net-(D29-A)
- U10 pad 2: +BATT -> Net-(D29-A)
- U10 pad 7: +BATT -> Net-(D29-A)
- U3 pad 12: +BATT -> Net-(D7-A)
- U3 pad 2: +BATT -> Net-(D7-A)
- U3 pad 7: +BATT -> Net-(D7-A)
- U6 pad 12: +BATT -> Net-(D15-A)
- U6 pad 2: +BATT -> Net-(D15-A)
- U6 pad 7: +BATT -> Net-(D15-A)
- U8 pad 12: +BATT -> Net-(D22-A)
- U8 pad 2: +BATT -> Net-(D22-A)
- U8 pad 7: +BATT -> Net-(D22-A)
Other:
- copper layers 2 -> 4

Commit message: Slight schematic adjustments and continue on draft pcb layout
Parts:
- removed J17: 01x05_Socket, Connector_PinSocket_2.54mm:PinSocket_1x05_P2.54mm_Vertical
- moved F3 197.9 mm to (138.0, 115.5)
- moved R83 190.4 mm to (104.5, 153.5)
- moved R87 190.4 mm to (104.5, 151.5)
- moved U6 190.4 mm to (112.5, 154.9)
- moved C19 187.5 mm to (66.5, 154.8)
- moved C20 187.5 mm to (67.0, 163.3)
- moved C22 187.5 mm to (78.0, 124.8)
- moved C24 187.5 mm to (96.3, 141.8)
- moved C26 187.5 mm to (67.5, 142.8)
- moved C27 187.5 mm to (72.5, 131.3)
- moved C28 187.5 mm to (78.5, 142.8)
- moved C46 187.5 mm to (121.5, 130.3)
- moved C83 187.5 mm to (82.0, 168.8)
- moved D10 187.5 mm to (92.5, 171.8)
- moved D11 187.5 mm to (80.0, 171.8)
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Connections:
- U2 pad 22: Net-(J17-Pin_5) -> unconnected-(U2-PC7-Pad22)
- U2 pad 23: Net-(J17-Pin_4) -> unconnected-(U2-PC6-Pad23)
- U2 pad 25: Net-(J17-Pin_3) -> unconnected-(U2-PC5-Pad25)
- U2 pad 26: Net-(J17-Pin_2) -> unconnected-(U2-PC4-Pad26)
- U2 pad 5: Net-(J17-Pin_1) -> unconnected-(U2-PC2-Pad5)

Commit message: Removed backups again, improved the PCB layout
Parts:
- Q11, Q12, Q13, Q14, Q15, Q16, Q17, Q18: moved to B.Cu
- moved C18 205.5 mm to (-135.0, 179.0)
- moved C19 205.5 mm to (-137.5, 179.0)
- moved C20 205.5 mm to (-137.0, 187.5)
- moved C21 205.5 mm to (-134.5, 187.5)
- moved C22 205.5 mm to (-126.0, 149.0)
- moved C24 205.5 mm to (-107.8, 166.0)
- moved C26 205.5 mm to (-136.5, 167.0)
- moved C27 205.5 mm to (-131.5, 155.5)
- moved C28 205.5 mm to (-125.5, 167.0)
- moved C46 205.5 mm to (-82.5, 154.5)
- moved C83 205.5 mm to (-122.0, 193.0)
- moved D10 205.5 mm to (-111.5, 196.0)
- moved D11 205.5 mm to (-124.0, 196.0)
- moved D12 205.5 mm to (-111.5, 173.5)
- moved D13 205.5 mm to (-124.5, 173.0)
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Routing:
- added copper zone on F.Cu, net +BATT
- added copper zone on F.Cu, net /Motor driver 4/MOT_SIDE_A
- added copper zone on F.Cu, net /Motor driver 4/MOT_SIDE_B
- added copper zone on F.Cu, net Net-(D32-K)
- added copper zone on F.Cu, net Net-(D33-A)

Commit message: Made layout of motor driver ch1, will replicate layout on other channels next.
Parts:
- moved R20 354.9 mm to (190.7, 109.9), turned to -90 degrees
- moved R86 353.5 mm to (194.0, 112.0), turned to -90 degrees
- moved R82 352.4 mm to (192.6, 112.0), turned to -90 degrees
- moved R19 351.6 mm to (190.7, 111.9), turned to -90 degrees
- moved R21 350.0 mm to (189.6, 111.9), turned to -90 degrees
- moved R18 346.6 mm to (185.5, 112.2), turned to -90 degrees
- moved C23 346.1 mm to (199.5, 124.5), turned to 0 degrees
- moved C17 344.2 mm to (190.5, 123.5)
- moved U3 343.5 mm to (191.0, 117.5), turned to -90 degrees
- moved C16 342.1 mm to (187.8, 111.9), turned to 90 degrees
- moved U4 339.4 mm to (197.0, 127.0), turned to 0 degrees
- moved C26 335.6 mm to (197.0, 129.8), turned to 180 degrees
- moved C19 335.0 mm to (193.0, 124.5), turned to 180 degrees
- moved R23 333.3 mm to (198.5, 132.5)
- moved R24 333.3 mm to (198.5, 131.5)
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Routing:
- net /Motor driver 1/MOT_SIDE_B: track 0.00 -> 62.8 mm, vias 0 -> 2
- net Net-(D7-A): track 0.00 -> 53.9 mm
- net /Motor driver 1/MOT_SIDE_A: track 0.00 -> 47.4 mm, vias 0 -> 1
- net Net-(D7-K): track 0.00 -> 40.4 mm
- net Net-(U3-AHO): track 0.00 -> 33.1 mm, vias 0 -> 4
- net Net-(U3-ALO): track 0.00 -> 27.2 mm, vias 0 -> 4
- net Net-(U3-BHO): track 0.00 -> 22.1 mm, vias 0 -> 4
- net Net-(D8-K): track 0.00 -> 21.6 mm
- net Net-(D11-A): track 0.00 -> 17.4 mm
- net Net-(U3-BLO): track 0.00 -> 14.8 mm, vias 0 -> 4
- net GND: track 0.00 -> 9.78 mm
- net Net-(U4-+): track 0.00 -> 6.38 mm
- net /Motor driver 1/LO_GATE_A: track 0.00 -> 6.29 mm
- net /Motor driver 1/LO_GATE_B: track 0.00 -> 5.12 mm
- net Net-(U3-DEL): track 0.00 -> 3.85 mm
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- added copper zone on B.Cu, net /Motor driver 1/MOT_SIDE_A
- added copper zone on F.Cu, net /Motor driver 1/MOT_SIDE_A
- added copper zone on B.Cu, net /Motor driver 1/MOT_SIDE_B
- added copper zone on F.Cu, net /Motor driver 1/MOT_SIDE_B
- added copper zone on F.Cu, net /Motor driver 2/MOT_SIDE_A
- added copper zone on F.Cu, net /Motor driver 2/MOT_SIDE_B
- added copper zone on F.Cu, net /Motor driver 3/MOT_SIDE_A
- added copper zone on F.Cu, net /Motor driver 3/MOT_SIDE_B
- added copper zone on B.Cu, net Net-(D10-K)
- added copper zone on F.Cu, net Net-(D10-K)
- added copper zone on B.Cu, net Net-(D11-A)
- added copper zone on F.Cu, net Net-(D11-A)
- added copper zone on B.Cu, net Net-(D18-K)
- added copper zone on F.Cu, net Net-(D18-K)
- added copper zone on B.Cu, net Net-(D19-A)
- added copper zone on F.Cu, net Net-(D19-A)
- added copper zone on B.Cu, net Net-(D25-K)
- added copper zone on F.Cu, net Net-(D25-K)
- added copper zone on B.Cu, net Net-(D26-A)
- added copper zone on F.Cu, net Net-(D26-A)
- added copper zone on B.Cu, net Net-(D32-K)
- added copper zone on B.Cu, net Net-(D33-A)
- added copper zone on F.Cu, net Net-(D7-A)

Commit message: Major PCB layout progress, motor drivers are routed and placed. PCB dimensions set, started ATMEGA2560 layout. Slight schematic fixes.
Parts:
- added G***: LOGO, Custom_feetprint:Fontys logo 12mm, F.Cu at (57.5, 97.0)
- added G***: LOGO, Custom_feetprint:fontys_aap_QR_15x15, B.Cu at (131.0, 111.0)
- moved J3 263.7 mm to (251.0, 139.9), turned to 90 degrees
- moved FB1 256.2 mm to (243.4, 134.6), turned to 180 degrees
- moved R5 251.2 mm to (245.0, 143.2)
- moved R6 249.0 mm to (242.0, 137.0), turned to 180 degrees
- moved R8 247.9 mm to (242.0, 140.7), turned to 0 degrees
- moved R7 247.9 mm to (242.0, 139.2), turned to 0 degrees
- moved D2 246.7 mm to (244.2, 131.5), turned to 0 degrees
- moved U12 246.3 mm to (242.0, 144.0)
- moved D6 243.5 mm to (246.0, 153.2), turned to 90 degrees
- moved C11 231.1 mm to (233.9, 137.1), turned to 0 degrees
- moved C82 229.9 mm to (234.6, 130.6), turned to -90 degrees
- moved C12 229.8 mm to (230.5, 142.3), turned to 90 degrees
- moved C14 226.1 mm to (233.0, 134.9), turned to 0 degrees
- moved JP1 225.1 mm to (231.1, 130.8), turned to -90 degrees
- moved R17 224.5 mm to (226.3, 144.9), turned to -90 degrees
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Routing:
- net /Motor driver 4/MOT_SIDE_B: track 0.00 -> 62.8 mm, vias 0 -> 2
- net /Motor driver 2/MOT_SIDE_B: track 0.00 -> 62.8 mm, vias 0 -> 2
- net /Motor driver 3/MOT_SIDE_B: track 0.00 -> 62.8 mm, vias 0 -> 2
- net Net-(D22-A): track 0.00 -> 53.9 mm
- net Net-(D15-A): track 0.00 -> 53.9 mm
- net /Motor driver 4/MOT_SIDE_A: track 0.00 -> 47.4 mm, vias 0 -> 1
- net /Motor driver 2/MOT_SIDE_A: track 0.00 -> 47.4 mm, vias 0 -> 1
- net /Motor driver 3/MOT_SIDE_A: track 0.00 -> 47.4 mm, vias 0 -> 1
- net Net-(D22-K): track 0.00 -> 40.4 mm
- net Net-(D15-K): track 0.00 -> 40.4 mm
- net Net-(D29-K): track 0.00 -> 38.2 mm
- net Net-(U8-AHO): track 0.00 -> 33.1 mm, vias 0 -> 4
- net Net-(U6-AHO): track 0.00 -> 33.1 mm, vias 0 -> 4
- net Net-(U10-AHO): track 0.00 -> 33.1 mm, vias 0 -> 4
- net /USB_GND: track 0.00 -> 28.1 mm, vias 0 -> 3
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- added copper zone on B.Cu, net GND
- added copper zone on F.Cu, net GND
- added copper zone on In1.Cu, net GND
- added copper zone on In2.Cu, net GND
- added copper zone on F.Cu, net Net-(D15-A)
- added copper zone on F.Cu, net Net-(D22-A)
- added copper zone on F.Cu, net Net-(D29-A)
- removed copper zone on B.Cu, net /Motor driver 1/MOT_SIDE_A
- removed copper zone on B.Cu, net /Motor driver 1/MOT_SIDE_B
- removed copper zone on B.Cu, net Net-(D10-K)
- removed copper zone on B.Cu, net Net-(D11-A)
- removed copper zone on B.Cu, net Net-(D18-K)
- removed copper zone on B.Cu, net Net-(D19-A)
- removed copper zone on B.Cu, net Net-(D25-K)
- removed copper zone on B.Cu, net Net-(D26-A)
- removed copper zone on B.Cu, net Net-(D32-K)
- removed copper zone on B.Cu, net Net-(D33-A)
Other:
- board outline added: 200 x 100 mm
- board text added: "Adaptive AGV platform"
- board text added: "Copyright © Mete Han Keskin, 2025 MIT License"
- board text added: "version V0.1"
