File: design_sources/KiCAD/controller_mainboard/dc_motor_driver.kicad_sch (KiCad schematic)
At the start: 45 parts, among them Q3 IRF3205, Q4 IRF3205, Q5 IRF3205, Q6 IRF3205, U3 HIP4082IBZT, U4 INA180A1IDBVR

Commit message: Changed JLCPCB field to LCSC
Parts:
- C16, C18, C19, C20, C21, C22, C24, C25: JLCPCB C15849 -> (none); LCSC (none) -> C15849
- C17, C23, C26, C28: JLCPCB C14663 -> (none); LCSC (none) -> C14663
- C27: JLCPCB C5246561 -> (none); LCSC (none) -> C5246561
- D10, D11, D12, D13, D7, D8: JLCPCB C22452 -> (none); LCSC (none) -> C22452
- D9: JLCPCB C2297 -> (none); LCSC (none) -> C2297
- L2, L3: JLCPCB C167953 -> (none); LCSC (none) -> C167953
- Q3, Q4, Q5, Q6: JLCPCB C2561 -> (none); LCSC (none) -> C2561
- R18, R19, R20, R21, R82, R86: JLCPCB C25744 -> (none); LCSC (none) -> C25744
- R22, R23, R24: JLCPCB C11702 -> (none); LCSC (none) -> C11702
- R25: JLCPCB C620706 -> (none); LCSC (none) -> C620706
- R64, R68, R72, R76: JLCPCB C21189 -> (none); LCSC (none) -> C21189
- U3: JLCPCB C50123 -> (none); LCSC (none) -> C50123
- U4: JLCPCB C122228 -> (none); LCSC (none) -> C122228
Changed lines of the file:
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@@
 			)
 		)
-		(property "JLCPCB" "C2561"
+		(property "LCSC" "C2561"
 			(at 179.07 76.2 0)
 			(effects
@@
 			)
 		)
-		(property "JLCPCB" "C21189"
-			(at 110.49 90.17 0)
+		(property "LCSC" "C21189"
+			(at 110.49 90.17 90)
 			(effects
 				(font
@@
 			)
 		)
-		(property "JLCPCB" "C15849"
+		(property "LCSC" "C15849"
 			(at 68.58 55.88 0)
 			(effects
@@
 			)
 		)
-		(property "JLCPCB" "C15849"
-			(at 134.62 85.09 0)
+		(property "LCSC" "C15849"
+			(at 134.62 85.09 90)
 			(effects
 				(font
@@
 			)
 		)
-		(property "JLCPCB" "C25744"
+		(property "LCSC" "C25744"
 			(at 57.15 92.71 0)
 			(effects
@@
 			)
 		)
-		(property "JLCPCB" "C14663"
+		(property "LCSC" "C14663"
 			(at 160.02 125.73 0)
 			(effects
@@
 			)
 		)
-		(property "JLCPCB" "C15849"
-			(at 134.62 73.66 0)
+		(property "LCSC" "C15849"
+			(at 134.62 73.66 90)
 			(effects
 				(font
@@
 			)
 		)
-		(property "JLCPCB" "C21189"
-			(at 110.49 111.76 0)
+		(property "LCSC" "C21189"
+			(at 110.49 111.76 90)
 			(effects
 				(font
@@
 			)
 		)
-		(property "JLCPCB" "C2561"
+		(property "LCSC" "C2561"
 			(at 241.3 76.2 0)
 			(effects
@@
 			)
 		)
-		(property "JLCPCB" "C50123"
+		(property "LCSC" "C50123"
 			(at 85.09 81.28 0)
 			(effects
@@
 			)
 		)
-		(property "JLCPCB" "C167953"
+		(property "LCSC" "C167953"
 			(at 147.32 39.37 90)
 			(effects
@@
 			)
 		)
-		(property "JLCPCB" "C15849"
+		(property "LCSC" "C15849"
 			(at 165.1 48.26 0)
 			(effects
@@
 			)
 		)
-		(property "JLCPCB" "C25744"
+		(property "LCSC" "C25744"
 			(at 68.58 107.95 0)
 			(effects
@@
 			)
 		)
-		(property "JLCPCB" "C21189"
-			(at 110.49 95.25 0)
+		(property "LCSC" "C21189"
+			(at 110.49 95.25 90)
 			(effects
 				(font
@@
 			)
 		)
-		(property "JLCPCB" "C22452"
+		(property "LCSC" "C22452"
 			(at 101.6 57.15 90)
 			(effects
@@
 			)
 		)
-		(property "JLCPCB" "C15849"
-			(at 134.62 80.01 0)
+		(property "LCSC" "C15849"
+			(at 134.62 80.01 90)
 			(effects
 				(font
@@
 			)
 		)
-		(property "JLCPCB" "C22452"
+		(property "LCSC" "C22452"
 			(at 195.58 101.6 90)
 			(effects
@@
 			)
 		)
-		(property "JLCPCB" "C620706"
+		(property "LCSC" "C620706"
 			(at 210.82 142.24 0)
 			(effects
@@
 			)
 		)
-		(property "JLCPCB" "C25744"
+		(property "LCSC" "C25744"
 			(at 34.29 76.2 0)
 			(effects
@@
 			)
 		)
-		(property "JLCPCB" "C25744"
+		(property "LCSC" "C25744"
 			(at 73.66 113.03 0)
 			(effects
@@
 			)
 		)
-		(property "JLCPCB" "C14663"
+		(property "LCSC" "C14663"
 			(at 233.68 142.24 0)
 			(effects
@@
 			)
 		)
-		(property "JLCPCB" "C25744"
+		(property "LCSC" "C25744"
 			(at 68.58 118.11 0)
 			(effects
@@
 			)
 		)
-		(property "JLCPCB" "C21189"
-			(at 110.49 116.84 0)
+		(property "LCSC" "C21189"
+			(at 110.49 116.84 90)
 			(effects
 				(font
@@
 			)
 		)
-		(property "JLCPCB" "C22452"
+		(property "LCSC" "C22452"
 			(at 195.58 76.2 90)
 			(effects
@@
 			)
 		)
-		(property "JLCPCB" "C15849"
+		(property "LCSC" "C15849"
 			(at 173.99 48.26 0)
 			(effects
@@
 			)
 		)
-		(property "JLCPCB" "C5246561"
+		(property "LCSC" "C5246561"
 			(at 182.88 48.26 0)
 			(effects
@@
 			)
 		)
-		(property "JLCPCB" "C22452"
+		(property "LCSC" "C22452"
 			(at 224.79 101.6 90)
 			(effects
@@
 			)
 		)
-		(property "JLCPCB" "C22452"
+		(property "LCSC" "C22452"
 			(at 106.68 57.15 90)
 			(effects
@@
 			)
 		)
-		(property "JLCPCB" "C25744"
+		(property "LCSC" "C25744"
 			(at 53.34 92.71 0)
 			(effects
@@
 			)
 		)
-		(property "JLCPCB" "C2297"
-			(at 121.92 55.88 0)
+		(property "LCSC" "C2297"
+			(at 121.92 55.88 90)
 			(effects
 				(font
@@
 			)
 		)
-		(property "JLCPCB" "C167953"
+		(property "LCSC" "C167953"
 			(at 147.32 44.45 90)
 			(effects
@@
 			)
 		)
-		(property "JLCPCB" "C11702"
-			(at 195.58 144.78 0)
+		(property "LCSC" "C11702"
+			(at 195.58 144.78 90)
 			(effects
 				(font
@@
 			)
 		)
-		(property "JLCPCB" "C14663"
+		(property "LCSC" "C14663"
 			(at 77.47 55.88 0)
 			(effects
@@
 			)
 		)
-		(property "JLCPCB" "C15849"
+		(property "LCSC" "C15849"
 			(at 137.16 48.26 0)
 			(effects
@@
 			)
 		)
-		(property "JLCPCB" "C2561"
+		(property "LCSC" "C2561"
 			(at 241.3 101.6 0)
 			(effects
@@
 			)
 		)
-		(property "JLCPCB" "C22452"
+		(property "LCSC" "C22452"
 			(at 224.79 76.2 90)
 			(effects
@@
 			)
 		)
-		(property "JLCPCB" "C15849"
-			(at 134.62 68.58 0)
+		(property "LCSC" "C15849"
+			(at 134.62 68.58 90)
 			(effects
 				(font
@@
 			)
 		)
-		(property "JLCPCB" "C122228"
+		(property "LCSC" "C122228"
 			(at 165.1 142.24 0)
 			(effects
@@
 			)
 		)
-		(property "JLCPCB" "C11702"
-			(at 195.58 139.7 0)
+		(property "LCSC" "C11702"
+			(at 195.58 139.7 90)
 			(effects
 				(font
@@
 			)
 		)
-		(property "JLCPCB" "C11702"
+		(property "LCSC" "C11702"
 			(at 121.92 46.99 0)
 			(effects
@@
 			)
 		)
-		(property "JLCPCB" "C14663"
+		(property "LCSC" "C14663"
 			(at 180.34 142.24 0)
 			(effects
@@
 			)
 		)
-		(property "JLCPCB" "C2561"
+		(property "LCSC" "C2561"
 			(at 179.07 101.6 0)
 			(effects

Commit message: Updated 50m750mW resistor lcsc mpn number, re-generated production files
Parts:
- R25: LCSC C620706 -> C127698
Changed lines of the file:
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@@
 			)
 		)
-		(property "LCSC" "C620706"
+		(property "LCSC" "C127698"
 			(at 210.82 142.24 0)
 			(effects
